Commit message: Fix typo & coherence

File: debra_description/urdf/arm_support.xacro (robot description, xacro)
@@ -1,4 +1,4 @@
 <?xml version="1.0"?>
-<robot name="wheel" xmlns:xacro="http://www.ros.org/wiki/xacro">
+<robot name="arm_support" xmlns:xacro="http://www.ros.org/wiki/xacro">
   <!-- Included URDF/XACRO Files -->
   <xacro:include

File: debra_description/urdf/common_properties.xacro (robot description, xacro)
@@ -3,6 +3,6 @@
   <!-- General properties -->
   <!--All units in m-kg-s-radians unit system -->
-  <property name="M_PI" value="3.1415926535897931" />
-  <property name="update_rate" value="10" />
+  <xacro:property name="M_PI" value="3.1415926535897931" />
+  <xacro:property name="update_rate" value="10" />
   <!-- Inertia -->
   <!-- Units are kg*m^2 -->
@@ -13,10 +13,10 @@
               izz="${m*(x*x+z*z)/12}" />
   </xacro:macro>
-  <macro name="cylinder_inertia"
-         params="m r h">
-    <inertia  ixx="${m*(3*r*r+h*h)/12}" ixy = "0" ixz = "0"
-              iyy="${m*(3*r*r+h*h)/12}" iyz = "0"
+  <xacro:macro name="cylinder_inertia"
+               params="m r h">
+    <inertia  ixx="${m*(3*r*r+h*h)/12}" ixy="0" ixz="0"
+              iyy="${m*(3*r*r+h*h)/12}" iyz="0"
               izz="${m*r*r/2}" />
-  </macro>
+  </xacro:macro>
   <!-- Base -->
   <xacro:property name="base_x_size" value="0.25" />
@@ -25,10 +25,10 @@
   <xacro:property name="base_mass" value="0.2" /> <!-- in kg-->
   <!-- Wheels -->
-  <property name="wheel_radius" value="0.03" />
-  <property name="wheel_height" value="0.01" />
-  <property name="wheel_mass" value="0.02" /> <!-- in kg -->
-  <property name="base_x_origin_to_wheel_origin" value="0.0" />
-  <property name="base_y_origin_to_wheel_origin" value="0.1" />
-  <property name="base_z_origin_to_wheel_origin" value="-0.01" />
+  <xacro:property name="wheel_radius" value="0.03" />
+  <xacro:property name="wheel_height" value="0.01" />
+  <xacro:property name="wheel_mass" value="0.02" /> <!-- in kg -->
+  <xacro:property name="base_x_origin_to_wheel_origin" value="0.0" />
+  <xacro:property name="base_y_origin_to_wheel_origin" value="0.1" />
+  <xacro:property name="base_z_origin_to_wheel_origin" value="-0.01" />
   <xacro:property name="wheel_separation"
                   value="${base_y_origin_to_wheel_origin * 2}" />
@@ -38,7 +38,7 @@
   <xacro:property name="arm_support_z_size" value="0.25" />
   <xacro:property name="arm_support_mass" value="0.1" />
-  <property name="arm_support_x_origin_to_wheel_origin" value="0.0" />
-  <property name="arm_support_y_origin_to_wheel_origin" value="0.1" />
-  <property name="arm_support_z_origin_to_wheel_origin"
-            value="${0.125 + base_z_size / 2}" />
+  <xacro:property name="arm_support_x_origin_to_wheel_origin" value="0.0" />
+  <xacro:property name="arm_support_y_origin_to_wheel_origin" value="0.1" />
+  <xacro:property name="arm_support_z_origin_to_wheel_origin"
+                  value="${0.125 + base_z_size / 2}" />
 </robot>

File: debra_description/urdf/debra.xacro (robot description, xacro)
@@ -12,5 +12,5 @@
       <mass value="0.0001" />
       <origin xyz="0 0 0"
-              rpy="0 0 0"/>
+              rpy="0 0 0" />
       <inertia ixx="0.0001" ixy="0.0" ixz="0.0"
                iyy="0.0001" iyz="0.0"

Commit message: Add arm slider part

File: debra_description/urdf/arm_support.xacro (robot description, xacro)
@@ -41,5 +41,5 @@
       <mu1 value="0.2"/>
       <mu2 value="0.2"/>
-      <material>Gazebo/Blue</material>
+      <material>Gazebo/Grey</material>
       <turnGravityOff>false</turnGravityOff>
     </gazebo>

File: debra_description/urdf/common_properties.xacro (robot description, xacro)
@@ -33,5 +33,5 @@
   <xacro:property name="wheel_separation"
                   value="${base_y_origin_to_wheel_origin * 2}" />
-    <!-- Arm support -->
+  <!-- Arm support -->
   <xacro:property name="arm_support_x_size" value="0.05" />
   <xacro:property name="arm_support_y_size" value="0.05" />
@@ -42,3 +42,12 @@
   <xacro:property name="arm_support_z_origin_to_wheel_origin"
                   value="${0.125 + base_z_size / 2}" />
+  <!-- Arm slider -->
+  <xacro:property name="arm_slider_x_size" value="${arm_support_x_size}" />
+  <xacro:property name="arm_slider_y_size" value="${arm_support_y_size}" />
+  <xacro:property name="arm_slider_z_size" value="0.02" />
+  <xacro:property name="arm_slider_mass" value="0.01" />
+  <xacro:property name="arm_slider_x_origin_to_wheel_origin" value="0.0" />
+  <xacro:property name="arm_slider_y_origin_to_wheel_origin"
+                  value="${(arm_support_y_size + arm_slider_y_size) / 2}" />
+  <xacro:property name="arm_slider_z_origin_to_wheel_origin" value="0.0" />
 </robot>

File: debra_description/urdf/debra.urdf (robot description, URDF)
Before this commit: robot debra, 6 links, 5 joints
Links:
- added link left_arm_slider, mass 0.01; collision box size=0.05 0.05 0.02; visual box size=0.05 0.05 0.02
- added link right_arm_slider, mass 0.01; collision box size=0.05 0.05 0.02; visual box size=0.05 0.05 0.02
Joints:
- added joint left_arm_slider_joint: type fixed, parent left_arm_support, child left_arm_slider, origin xyz=0.0                    0.05                    0.0 rpy=0 0 0
- added joint right_arm_slider_joint: type fixed, parent right_arm_support, child right_arm_slider, origin xyz=0.0                    -0.05                    0.0 rpy=0 0 0

File: debra_description/urdf/debra.xacro (robot description, xacro)
@@ -6,4 +6,5 @@
   <xacro:include filename="$(find debra_description)/urdf/wheel.xacro" />
   <xacro:include filename="$(find debra_description)/urdf/arm_support.xacro" />
+  <xacro:include filename="$(find debra_description)/urdf/arm_slider.xacro" />
   <!-- BASE-FOOTPRINT -->
   <!-- base_footprint is a fictitious link(frame) that is on the ground right below base_link origin -->
@@ -12,5 +13,5 @@
       <mass value="0.0001" />
       <origin xyz="0 0 0"
-              rpy="0 0 0" />
+              rpy="0 0 0"/>
       <inertia ixx="0.0001" ixy="0.0" ixz="0.0"
                iyy="0.0001" iyz="0.0"
@@ -93,4 +94,14 @@
                translateY="1"
                flipY="0" />
+  <arm_slider lr="right"
+              parent="right_arm_support"
+              translateX="1"
+              translateY="-1"
+              flipY="0" />
+  <arm_slider lr="left"
+              parent="left_arm_support"
+              translateX="1"
+              translateY="1"
+              flipY="0" />
   <gazebo>
     <plugin name="differential_drive_controller"
