Commit message: Solve controller calls errors

File: debra_description/urdf/arm_slider.xacro (robot description, xacro)
@@ -45,8 +45,12 @@
     </gazebo>
     <joint name="${lr}_arm_slider_joint"
-           type="fixed">
+           type="prismatic">
       <parent link="${parent}"/>
       <child link="${lr}_arm_slider"/>
       <hardwareInterface>EffortJointInterface</hardwareInterface>
+      <limit effort="1000.0"
+             lower="-0.38"
+             upper="0"
+             velocity="0.5" />
       <origin xyz="${translateX * arm_slider_x_origin_to_wheel_origin}
                    ${translateY * arm_slider_y_origin_to_wheel_origin}
@@ -54,4 +58,13 @@
               rpy="0 0 0" />
     </joint>
+    <!-- Transmission is important to link the joints and the controller -->
+    <transmission name="${parent}_${lr}_arm_slider_joint_trans">
+      <type>transmission_interface/SimpleTransmission</type>
+      <joint name="${parent}_${lr}_arm_slider_joint" />
+      <actuator name="${parent}_${lr}_arm_slider_joint_motor">
+        <hardwareInterface>EffortJointInterface</hardwareInterface>
+        <mechanicalReduction>1</mechanicalReduction>
+      </actuator>
+    </transmission>
   </xacro:macro>
 </robot>

File: debra_description/urdf/debra.urdf (robot description, URDF)
Before this commit: robot debra, 8 links, 7 joints
Joints:
- joint left_arm_slider_joint: limit (none) -> lower=-0.38 upper=0 effort=1000.0 velocity=0.5; type fixed -> prismatic
- joint right_arm_slider_joint: limit (none) -> lower=-0.38 upper=0 effort=1000.0 velocity=0.5; type fixed -> prismatic

Commit message: Fix errors in DOF & controller names

File: debra_description/urdf/arm_slider.xacro (robot description, xacro)
@@ -4,5 +4,4 @@
   <xacro:include
     filename="$(find debra_description)/urdf/common_properties.xacro" />
-  <!-- Wheels -->
   <xacro:macro name="arm_slider"
                params="lr parent translateX translateY flipY">
@@ -44,16 +43,18 @@
       <turnGravityOff>false</turnGravityOff>
     </gazebo>
-    <joint name="${lr}_arm_slider_joint"
+    <joint name="${parent}_${lr}_arm_slider_joint"
            type="prismatic">
       <parent link="${parent}"/>
       <child link="${lr}_arm_slider"/>
       <hardwareInterface>EffortJointInterface</hardwareInterface>
+      <axis xyz="0 0 1"
+            rpy="0 0 0" />
       <limit effort="1000.0"
-             lower="-0.38"
-             upper="0"
+             lower="${arm_slider_limit_lower}"
+             upper="${arm_slider_limit_upper}"
              velocity="0.5" />
-      <origin xyz="${translateX * arm_slider_x_origin_to_wheel_origin}
-                   ${translateY * arm_slider_y_origin_to_wheel_origin}
-                   ${arm_slider_z_origin_to_wheel_origin}"
+      <origin xyz="${translateX * arm_slider_x_origin_to_base_origin}
+                   ${translateY * arm_slider_y_origin_to_base_origin}
+                   ${arm_slider_z_origin_to_base_origin}"
               rpy="0 0 0" />
     </joint>
@@ -61,5 +62,7 @@
     <transmission name="${parent}_${lr}_arm_slider_joint_trans">
       <type>transmission_interface/SimpleTransmission</type>
-      <joint name="${parent}_${lr}_arm_slider_joint" />
+      <joint name="${parent}_${lr}_arm_slider_joint">
+        <hardwareInterface>EffortJointInterface</hardwareInterface>
+      </joint>
       <actuator name="${parent}_${lr}_arm_slider_joint_motor">
         <hardwareInterface>EffortJointInterface</hardwareInterface>

File: debra_description/urdf/arm_support.xacro (robot description, xacro)
@@ -4,5 +4,4 @@
   <xacro:include
     filename="$(find debra_description)/urdf/common_properties.xacro" />
-  <!-- Wheels -->
   <xacro:macro name="arm_support"
                params="lr parent translateX translateY flipY">
@@ -49,7 +48,7 @@
       <child link="${lr}_arm_support"/>
       <hardwareInterface>EffortJointInterface</hardwareInterface>
-      <origin xyz="${translateX * arm_support_x_origin_to_wheel_origin}
-                   ${translateY * arm_support_y_origin_to_wheel_origin}
-                   ${arm_support_z_origin_to_wheel_origin}"
+      <origin xyz="${translateX * arm_support_x_origin_to_base_origin}
+                   ${translateY * arm_support_y_origin_to_base_origin}
+                   ${arm_support_z_origin_to_base_origin}"
               rpy="0 0 0" />
     </joint>

File: debra_description/urdf/common_properties.xacro (robot description, xacro)
@@ -1,4 +1,4 @@
 <?xml version="1.0"?>
-<robot name="wheel" xmlns:xacro="http://www.ros.org/wiki/xacro">
+<robot name="common_properties" xmlns:xacro="http://www.ros.org/wiki/xacro">
   <!-- General properties -->
   <!--All units in m-kg-s-radians unit system -->
@@ -33,21 +33,24 @@
   <xacro:property name="wheel_separation"
                   value="${base_y_origin_to_wheel_origin * 2}" />
-  <!-- Arm support -->
+  <!-- Arm supports -->
   <xacro:property name="arm_support_x_size" value="0.05" />
   <xacro:property name="arm_support_y_size" value="0.05" />
   <xacro:property name="arm_support_z_size" value="0.25" />
   <xacro:property name="arm_support_mass" value="0.1" />
-  <xacro:property name="arm_support_x_origin_to_wheel_origin" value="0.0" />
-  <xacro:property name="arm_support_y_origin_to_wheel_origin" value="0.1" />
-  <xacro:property name="arm_support_z_origin_to_wheel_origin"
+  <xacro:property name="arm_support_x_origin_to_base_origin" value="0.0" />
+  <xacro:property name="arm_support_y_origin_to_base_origin" value="0.1" />
+  <xacro:property name="arm_support_z_origin_to_base_origin"
                   value="${0.125 + base_z_size / 2}" />
-  <!-- Arm slider -->
+  <!-- Arm sliders -->
   <xacro:property name="arm_slider_x_size" value="${arm_support_x_size}" />
   <xacro:property name="arm_slider_y_size" value="${arm_support_y_size}" />
   <xacro:property name="arm_slider_z_size" value="0.02" />
   <xacro:property name="arm_slider_mass" value="0.01" />
-  <xacro:property name="arm_slider_x_origin_to_wheel_origin" value="0.0" />
-  <xacro:property name="arm_slider_y_origin_to_wheel_origin"
+  <xacro:property name="arm_slider_x_origin_to_base_origin" value="0.0" />
+  <xacro:property name="arm_slider_y_origin_to_base_origin"
                   value="${(arm_support_y_size + arm_slider_y_size) / 2}" />
-  <xacro:property name="arm_slider_z_origin_to_wheel_origin" value="0.0" />
+  <xacro:property name="arm_slider_z_origin_to_base_origin"
+                  value="${(arm_support_z_size - arm_slider_z_size) / 2}" />
+  <xacro:property name="arm_slider_limit_upper" value="0.3" />
+  <xacro:property name="arm_slider_limit_lower" value="0" />
 </robot>

File: debra_description/urdf/debra.urdf (robot description, URDF)
Before this commit: robot debra, 8 links, 7 joints
Links:
- link base_footprint: mass 0.0001 -> None
Joints:
- removed joint left_arm_slider_joint
- removed joint right_arm_slider_joint
- added joint left_arm_support_left_arm_slider_joint: type prismatic, parent left_arm_support, child left_arm_slider, origin xyz=0.0                    0.05                    0.115 rpy=0 0 0, axis 0 0 1, limit lower=0 upper=0.3 effort=1000.0 velocity=0.5
- added joint right_arm_support_right_arm_slider_joint: type prismatic, parent right_arm_support, child right_arm_slider, origin xyz=0.0                    -0.05                    0.115 rpy=0 0 0, axis 0 0 1, limit lower=0 upper=0.3 effort=1000.0 velocity=0.5

File: debra_description/urdf/debra.xacro (robot description, xacro)
@@ -10,12 +10,4 @@
   <!-- base_footprint is a fictitious link(frame) that is on the ground right below base_link origin -->
   <link name="base_footprint">
-    <inertial>
-      <mass value="0.0001" />
-      <origin xyz="0 0 0"
-              rpy="0 0 0"/>
-      <inertia ixx="0.0001" ixy="0.0" ixz="0.0"
-               iyy="0.0001" iyz="0.0"
-               izz="0.0001" />
-    </inertial>
     <visual>
         <origin xyz="0 0 0"
@@ -104,4 +96,5 @@
               translateY="1"
               flipY="0" />
+  <!-- Base controller -->
   <gazebo>
     <plugin name="differential_drive_controller"
@@ -122,10 +115,17 @@
             filename="libgazebo_ros_control.so" />
   </gazebo>
-    <!-- Hokuyo laser -->
+  <!-- Arm controller -->
+  <gazebo>
+    <plugin name="gazebo_ros_control"
+            filename="libgazebo_ros_control.so">
+      <robotNamespace>/debra</robotNamespace>
+    </plugin>
+  </gazebo>
+    <!-- Hokuyo laser controller -->
   <gazebo reference="hokuyo_link">
     <sensor type="gpu_ray" name="head_hokuyo_sensor">
       <pose>0 0 0 0 0 0</pose>
       <visualize>false</visualize>
-      <update_rate>40</update_rate>
+      <update_rate>50</update_rate>
       <ray>
         <scan>
@@ -153,5 +153,5 @@
       </ray>
       <plugin name="gazebo_ros_head_hokuyo_controller" filename="libgazebo_ros_gpu_laser.so">
-        <topicName>/rrbot/laser/scan</topicName>
+        <topicName>/debra/laser/scan</topicName>
         <frameName>hokuyo_link</frameName>
       </plugin>

File: debra_description/urdf/wheel.xacro (robot description, xacro)
@@ -62,5 +62,7 @@
     <transmission name="${parent}_${lr}_wheel_joint_trans">
       <type>transmission_interface/SimpleTransmission</type>
-      <joint name="${parent}_${lr}_wheel_joint" />
+      <joint name="${parent}_${lr}_wheel_joint">
+        <hardwareInterface>EffortJointInterface</hardwareInterface>
+      </joint>
       <actuator name="${parent}_${lr}_wheel_joint_motor">
         <hardwareInterface>EffortJointInterface</hardwareInterface>
