Commit message: Add arm support as link fixed to base

File: debra_description/urdf/common_properties.xacro (robot description, xacro)
@@ -5,9 +5,5 @@
   <property name="M_PI" value="3.1415926535897931" />
   <property name="update_rate" value="10" />
-  <!-- Base -->
-  <xacro:property name="base_x_size" value="0.5" />
-  <xacro:property name="base_y_size" value="0.5" />
-  <xacro:property name="base_z_size" value="0.2" />
-  <xacro:property name="base_mass" value="1" /> <!-- in kg-->
+  <!-- Inertia -->
   <!-- Units are kg*m^2 -->
   <xacro:macro name="box_inertia"
@@ -17,14 +13,4 @@
               izz="${m*(x*x+z*z)/12}" />
   </xacro:macro>
-  <!-- Wheels -->
-  <property name="wheel_radius" value="0.2" />
-  <property name="wheel_height" value="0.05" />
-  <property name="wheel_mass" value="0.1" /> <!-- in kg -->
-  <property name="base_x_origin_to_wheel_origin" value="0.0" />
-  <property name="base_y_origin_to_wheel_origin" value="0.3" />
-  <property name="base_z_origin_to_wheel_origin" value="-0.1" />
-  <xacro:property name="wheel_separation"
-                  value="${base_y_origin_to_wheel_origin * 2}" />
-  <!-- Units are kg*m^2 -->
   <macro name="cylinder_inertia"
          params="m r h">
@@ -33,3 +19,26 @@
               izz="${m*r*r/2}" />
   </macro>
+  <!-- Base -->
+  <xacro:property name="base_x_size" value="0.25" />
+  <xacro:property name="base_y_size" value="0.25" />
+  <xacro:property name="base_z_size" value="0.05" />
+  <xacro:property name="base_mass" value="0.2" /> <!-- in kg-->
+  <!-- Wheels -->
+  <property name="wheel_radius" value="0.03" />
+  <property name="wheel_height" value="0.01" />
+  <property name="wheel_mass" value="0.02" /> <!-- in kg -->
+  <property name="base_x_origin_to_wheel_origin" value="0.0" />
+  <property name="base_y_origin_to_wheel_origin" value="0.1" />
+  <property name="base_z_origin_to_wheel_origin" value="-0.01" />
+  <xacro:property name="wheel_separation"
+                  value="${base_y_origin_to_wheel_origin * 2}" />
+    <!-- Arm support -->
+  <xacro:property name="arm_support_x_size" value="0.05" />
+  <xacro:property name="arm_support_y_size" value="0.05" />
+  <xacro:property name="arm_support_z_size" value="0.25" />
+  <xacro:property name="arm_support_mass" value="0.1" />
+  <property name="arm_support_x_origin_to_wheel_origin" value="0.0" />
+  <property name="arm_support_y_origin_to_wheel_origin" value="0.1" />
+  <property name="arm_support_z_origin_to_wheel_origin"
+            value="${0.125 + base_z_size / 2}" />
 </robot>

File: debra_description/urdf/debra.urdf (robot description, URDF)
Before this commit: robot debra, 4 links, 3 joints
Links:
- added link left_arm_support, mass 0.1; collision box size=0.05 0.05 0.25; visual box size=0.05 0.05 0.25
- added link right_arm_support, mass 0.1; collision box size=0.05 0.05 0.25; visual box size=0.05 0.05 0.25
- link base_link: mass 1 -> 0.2; geometry collision box size=0.25 0.25 0.05; visual box size=0.25 0.25 0.05
- link base_link_left_wheel: mass 0.1 -> 0.02; geometry collision cylinder length=0.01 radius=0.03; visual cylinder length=0.01 radius=0.03
- link base_link_right_wheel: mass 0.1 -> 0.02; geometry collision cylinder length=0.01 radius=0.03; visual cylinder length=0.01 radius=0.03
Joints:
- added joint left_arm_support_joint: type fixed, parent base_link, child left_arm_support, origin xyz=0.0                    0.1                    0.15 rpy=0 0 0
- added joint right_arm_support_joint: type fixed, parent base_link, child right_arm_support, origin xyz=0.0                    -0.1                    0.15 rpy=0 0 0
- joint base_footprint_joint: origin xyz=0 0 0.3 rpy=0 0 0 -> xyz=0 0 0.04 rpy=0 0 0
- joint base_link_left_wheel_joint: origin xyz=0.0                    0.3                    -0.1 rpy=0 0 0 -> xyz=0.0                    0.1                    -0.01 rpy=0 0 0
- joint base_link_right_wheel_joint: origin xyz=0.0                    -0.3                    -0.1 rpy=0 0 0 -> xyz=0.0                    -0.1                    -0.01 rpy=0 0 0

File: debra_description/urdf/debra.xacro (robot description, xacro)
@@ -5,4 +5,5 @@
   <xacro:include filename="$(find debra_description)/urdf/materials.xacro" />
   <xacro:include filename="$(find debra_description)/urdf/wheel.xacro" />
+  <xacro:include filename="$(find debra_description)/urdf/arm_support.xacro" />
   <!-- BASE-FOOTPRINT -->
   <!-- base_footprint is a fictitious link(frame) that is on the ground right below base_link origin -->
@@ -52,7 +53,7 @@
               rpy="0 0 0" />
       <geometry>
-        <box size="1 0.5 0.25"/>
+        <box size="${base_x_size} ${base_y_size} ${base_z_size}"/>
       </geometry>
-      <material name="Yellow" />
+      <material name="LightGrey" />
     </visual>
     <collision>
@@ -60,10 +61,12 @@
               rpy="0 0 0 " />
       <geometry>
-        <box size="1 0.5 0.25"/>
+        <box size="${base_x_size} ${base_y_size} ${base_z_size}"/>
       </geometry>
     </collision>
   </link>
   <gazebo reference="base_link">
-    <material>Gazebo/Yellow</material>
+    <mu1>0.2</mu1>
+    <mu2>0.2</mu2>
+    <material>Gazebo/White</material>
     <turnGravityOff>false</turnGravityOff>
   </gazebo>
@@ -73,10 +76,21 @@
          translateX="1"
          translateY="-1"
-         flipY="-1"/>
+         flipY="-1" />
   <wheel lr="left"
          parent="base_link"
          translateX="1"
          translateY="1"
-         flipY="-1"/>
+         flipY="-1" />
+  <!-- ARMS -->
+  <arm_support lr="right"
+               parent="base_link"
+               translateX="1"
+               translateY="-1"
+               flipY="0" />
+  <arm_support lr="left"
+               parent="base_link"
+               translateX="1"
+               translateY="1"
+               flipY="0" />
   <gazebo>
     <plugin name="differential_drive_controller"
@@ -97,3 +111,39 @@
             filename="libgazebo_ros_control.so" />
   </gazebo>
+    <!-- Hokuyo laser -->
+  <gazebo reference="hokuyo_link">
+    <sensor type="gpu_ray" name="head_hokuyo_sensor">
+      <pose>0 0 0 0 0 0</pose>
+      <visualize>false</visualize>
+      <update_rate>40</update_rate>
+      <ray>
+        <scan>
+          <horizontal>
+            <samples>720</samples>
+            <resolution>1</resolution>
+            <min_angle>-1.570796</min_angle>
+            <max_angle>1.570796</max_angle>
+          </horizontal>
+        </scan>
+        <range>
+          <min>0.10</min>
+          <max>30.0</max>
+          <resolution>0.01</resolution>
+        </range>
+        <noise>
+          <type>gaussian</type>
+          <!-- Noise parameters based on published spec for Hokuyo laser
+               achieving "+-30mm" accuracy at range < 10m.  A mean of 0.0m and
+               stddev of 0.01m will put 99.7% of samples within 0.03m of the
+               true reading. -->
+          <mean>0.0</mean>
+          <stddev>0.01</stddev>
+        </noise>
+      </ray>
+      <plugin name="gazebo_ros_head_hokuyo_controller" filename="libgazebo_ros_gpu_laser.so">
+        <topicName>/rrbot/laser/scan</topicName>
+        <frameName>hokuyo_link</frameName>
+      </plugin>
+    </sensor>
+  </gazebo>
 </robot>

File: debra_description/urdf/materials.xacro (robot description, xacro)
@@ -10,4 +10,7 @@
     <color rgba="0.0 0.8 0.0 1.0"/>
   </material>
+  <material name="LightLightGrey">
+    <color rgba="0.9 0.9 0.9 1.0"/>
+  </material>
   <material name="LightGrey">
     <color rgba="0.7 0.7 0.7 1.0"/>
@@ -18,4 +21,13 @@
   <material name="DarkGrey">
     <color rgba="0.3 0.3 0.3 1.0"/>
+  </material>
+  <material name="DarkDarkGrey">
+    <color rgba="0.1 0.1 0.1 1.0"/>
+  </material>
+  <material name="Orange">
+    <color rgba="${255/255} ${108/255} ${10/255} 1.0"/>
+  </material>
+  <material name="Brown">
+    <color rgba="${222/255} ${207/255} ${195/255} 1.0"/>
   </material>
   <material name="Red">

File: debra_description/urdf/wheel.xacro (robot description, xacro)
@@ -40,5 +40,5 @@
       <kd  value="1.0" />
       <fdir1 value="1 0 0"/>
-      <material>Gazebo/Grey</material>
+      <material>Gazebo/Blue</material>
       <turnGravityOff>false</turnGravityOff>
     </gazebo>

Commit message: Add arm link & shoulder joint

File: debra_description/urdf/common_properties.xacro (robot description, xacro)
@@ -54,3 +54,15 @@
   <xacro:property name="arm_slider_limit_upper" value="0.3" />
   <xacro:property name="arm_slider_limit_lower" value="0" />
+  <!-- Arm arms -->
+  <xacro:property name="arm_arm_x_size" value="0.04" />
+  <xacro:property name="arm_arm_y_size" value="0.15" />
+  <xacro:property name="arm_arm_z_size" value="0.03" />
+  <xacro:property name="arm_arm_mass" value="0.1" />
+  <xacro:property name="arm_arm_x_origin_to_base_origin" value="0.0" />
+  <xacro:property name="arm_arm_y_origin_to_base_origin"
+                  value="${(arm_arm_y_size - arm_slider_y_size) / 2 + 0.015}" />
+  <xacro:property name="arm_arm_z_origin_to_base_origin"
+                  value="${- (arm_slider_z_size + arm_arm_z_size) / 2}" />
+  <xacro:property name="arm_arm_limit_upper" value="${M_PI / 4}" />
+  <xacro:property name="arm_arm_limit_lower" value="${- M_PI / 4}" />
 </robot>

File: debra_description/urdf/debra.urdf (robot description, URDF)
Before this commit: robot debra, 8 links, 7 joints
Links:
- added link left_arm_arm, mass 0.1; collision box size=0.04 0.15 0.03; visual box size=0.04 0.15 0.03
- added link right_arm_arm, mass 0.1; collision box size=0.04 0.15 0.03; visual box size=0.04 0.15 0.03
Joints:
- added joint left_arm_slider_left_arm_arm_joint: type revolute, parent left_arm_slider, child left_arm_arm, origin xyz=0.0                    0.065                    -0.025 rpy=0 0 0, axis 0 0 1, limit lower=-0.785398163397 upper=0.785398163397 effort=1000.0 velocity=0.5
- added joint right_arm_slider_right_arm_arm_joint: type revolute, parent right_arm_slider, child right_arm_arm, origin xyz=0.0                    -0.065                    -0.025 rpy=0 0 0, axis 0 0 1, limit lower=-0.785398163397 upper=0.785398163397 effort=1000.0 velocity=0.5

File: debra_description/urdf/debra.xacro (robot description, xacro)
@@ -7,4 +7,5 @@
   <xacro:include filename="$(find debra_description)/urdf/arm_support.xacro" />
   <xacro:include filename="$(find debra_description)/urdf/arm_slider.xacro" />
+  <xacro:include filename="$(find debra_description)/urdf/arm_arm.xacro" />
   <!-- BASE-FOOTPRINT -->
   <!-- base_footprint is a fictitious link(frame) that is on the ground right below base_link origin -->
@@ -78,22 +79,32 @@
   <arm_support lr="right"
                parent="base_link"
-               translateX="1"
+               translateX="0"
                translateY="-1"
                flipY="0" />
   <arm_support lr="left"
                parent="base_link"
-               translateX="1"
+               translateX="0"
                translateY="1"
                flipY="0" />
   <arm_slider lr="right"
               parent="right_arm_support"
-              translateX="1"
+              translateX="0"
               translateY="-1"
               flipY="0" />
   <arm_slider lr="left"
               parent="left_arm_support"
-              translateX="1"
+              translateX="0"
               translateY="1"
               flipY="0" />
+  <arm_arm lr="right"
+           parent="right_arm_slider"
+           translateX="1"
+           translateY="-1"
+           flipY="0" />
+  <arm_arm lr="left"
+           parent="left_arm_slider"
+           translateX="1"
+           translateY="1"
+           flipY="0" />
   <!-- Base controller -->
   <gazebo>

Commit message: Add forearm link & elbow joint

File: debra_description/urdf/common_properties.xacro (robot description, xacro)
@@ -56,13 +56,25 @@
   <!-- Arm arms -->
   <xacro:property name="arm_arm_x_size" value="0.04" />
-  <xacro:property name="arm_arm_y_size" value="0.15" />
+  <xacro:property name="arm_arm_y_size" value="0.20" />
   <xacro:property name="arm_arm_z_size" value="0.03" />
   <xacro:property name="arm_arm_mass" value="0.1" />
   <xacro:property name="arm_arm_x_origin_to_base_origin" value="0.0" />
   <xacro:property name="arm_arm_y_origin_to_base_origin"
-                  value="${(arm_arm_y_size - arm_slider_y_size) / 2 + 0.015}" />
+                  value="${(arm_arm_y_size + arm_slider_y_size) / 2 - 0.04}" />
   <xacro:property name="arm_arm_z_origin_to_base_origin"
                   value="${- (arm_slider_z_size + arm_arm_z_size) / 2}" />
   <xacro:property name="arm_arm_limit_upper" value="${M_PI / 4}" />
   <xacro:property name="arm_arm_limit_lower" value="${- M_PI / 4}" />
+  <!-- Arm forearms -->
+  <xacro:property name="arm_forearm_x_size" value="0.04" />
+  <xacro:property name="arm_forearm_y_size" value="0.20" />
+  <xacro:property name="arm_forearm_z_size" value="0.03" />
+  <xacro:property name="arm_forearm_mass" value="0.1" />
+  <xacro:property name="arm_forearm_x_origin_to_base_origin" value="0.0" />
+  <xacro:property name="arm_forearm_y_origin_to_base_origin"
+                  value="${(arm_arm_y_size + arm_forearm_y_size) / 2 - 0.04}" />
+  <xacro:property name="arm_forearm_z_origin_to_base_origin"
+                  value="${- (arm_arm_z_size + arm_forearm_z_size) / 2}" />
+  <xacro:property name="arm_forearm_limit_upper" value="${M_PI / 4}" />
+  <xacro:property name="arm_forearm_limit_lower" value="${- M_PI / 4}" />
 </robot>

File: debra_description/urdf/debra.urdf (robot description, URDF)
Before this commit: robot debra, 10 links, 9 joints
Links:
- added link left_arm_forearm, mass 0.1; collision box size=0.04 0.2 0.03; visual box size=0.04 0.2 0.03
- added link right_arm_forearm, mass 0.1; collision box size=0.04 0.2 0.03; visual box size=0.04 0.2 0.03
- link left_arm_arm: geometry collision box size=0.04 0.2 0.03; visual box size=0.04 0.2 0.03
- link right_arm_arm: geometry collision box size=0.04 0.2 0.03; visual box size=0.04 0.2 0.03
Joints:
- added joint left_arm_arm_left_arm_forearm_joint: type revolute, parent left_arm_arm, child left_arm_forearm, origin xyz=0.0                    0.16                    -0.03 rpy=0 0 0, axis 0 0 1, limit lower=-0.785398163397 upper=0.785398163397 effort=1000.0 velocity=0.5
- added joint right_arm_arm_right_arm_forearm_joint: type revolute, parent right_arm_arm, child right_arm_forearm, origin xyz=0.0                    -0.16                    -0.03 rpy=0 0 0, axis 0 0 1, limit lower=-0.785398163397 upper=0.785398163397 effort=1000.0 velocity=0.5
- joint left_arm_slider_left_arm_arm_joint: origin xyz=0.0                    0.065                    -0.025 rpy=0 0 0 -> xyz=0.0                    0.085                    -0.025 rpy=0 0 0
- joint right_arm_slider_right_arm_arm_joint: origin xyz=0.0                    -0.065                    -0.025 rpy=0 0 0 -> xyz=0.0                    -0.085                    -0.025 rpy=0 0 0

File: debra_description/urdf/debra.xacro (robot description, xacro)
@@ -8,4 +8,5 @@
   <xacro:include filename="$(find debra_description)/urdf/arm_slider.xacro" />
   <xacro:include filename="$(find debra_description)/urdf/arm_arm.xacro" />
+  <xacro:include filename="$(find debra_description)/urdf/arm_forearm.xacro" />
   <!-- BASE-FOOTPRINT -->
   <!-- base_footprint is a fictitious link(frame) that is on the ground right below base_link origin -->
@@ -99,12 +100,22 @@
   <arm_arm lr="right"
            parent="right_arm_slider"
-           translateX="1"
+           translateX="0"
            translateY="-1"
            flipY="0" />
   <arm_arm lr="left"
            parent="left_arm_slider"
-           translateX="1"
+           translateX="0"
            translateY="1"
            flipY="0" />
+  <arm_forearm lr="right"
+               parent="right_arm_arm"
+               translateX="0"
+               translateY="-1"
+               flipY="0" />
+  <arm_forearm lr="left"
+               parent="left_arm_arm"
+               translateX="0"
+               translateY="1"
+               flipY="0" />
   <!-- Base controller -->
   <gazebo>

Commit message: Replace arm support links w/ a single body link

File: debra_description/urdf/common_properties.xacro (robot description, xacro)
@@ -23,5 +23,15 @@
   <xacro:property name="base_y_size" value="0.25" />
   <xacro:property name="base_z_size" value="0.05" />
-  <xacro:property name="base_mass" value="0.2" /> <!-- in kg-->
+  <xacro:property name="base_mass" value="0.5" /> <!-- in kg-->
+  <!-- Body -->
+  <xacro:property name="body_x_size" value="0.08" />
+  <xacro:property name="body_y_size"
+                  value="${base_y_size - 2 * arm_slider_y_size}" />
+  <xacro:property name="body_z_size" value="0.30" />
+  <xacro:property name="body_mass" value="0.2" />
+  <xacro:property name="body_x_origin_to_base_origin" value="0.0" />
+  <xacro:property name="body_y_origin_to_base_origin" value="0.0" />
+  <xacro:property name="body_z_origin_to_base_origin"
+                  value="${(body_z_size + base_z_size) / 2}" />
   <!-- Wheels -->
   <xacro:property name="wheel_radius" value="0.03" />
@@ -33,25 +43,17 @@
   <xacro:property name="wheel_separation"
                   value="${base_y_origin_to_wheel_origin * 2}" />
-  <!-- Arm supports -->
-  <xacro:property name="arm_support_x_size" value="0.05" />
-  <xacro:property name="arm_support_y_size" value="0.05" />
-  <xacro:property name="arm_support_z_size" value="0.25" />
-  <xacro:property name="arm_support_mass" value="0.1" />
-  <xacro:property name="arm_support_x_origin_to_base_origin" value="0.0" />
-  <xacro:property name="arm_support_y_origin_to_base_origin" value="0.1" />
-  <xacro:property name="arm_support_z_origin_to_base_origin"
-                  value="${0.125 + base_z_size / 2}" />
   <!-- Arm sliders -->
-  <xacro:property name="arm_slider_x_size" value="${arm_support_x_size}" />
-  <xacro:property name="arm_slider_y_size" value="${arm_support_y_size}" />
+  <xacro:property name="arm_slider_x_size" value="0.05" />
+  <xacro:property name="arm_slider_y_size" value="0.05" />
   <xacro:property name="arm_slider_z_size" value="0.02" />
   <xacro:property name="arm_slider_mass" value="0.01" />
   <xacro:property name="arm_slider_x_origin_to_base_origin" value="0.0" />
   <xacro:property name="arm_slider_y_origin_to_base_origin"
-                  value="${(arm_support_y_size + arm_slider_y_size) / 2}" />
+                  value="${(body_y_size + arm_slider_y_size) / 2}" />
   <xacro:property name="arm_slider_z_origin_to_base_origin"
-                  value="${(arm_support_z_size - arm_slider_z_size) / 2}" />
-  <xacro:property name="arm_slider_limit_upper" value="0.3" />
-  <xacro:property name="arm_slider_limit_lower" value="0" />
+                  value="${(body_z_size - arm_slider_z_size) / 2}" />
+  <xacro:property name="arm_slider_limit_upper" value="0.0" />
+  <xacro:property name="arm_slider_limit_lower"
+                  value="${- body_z_size + arm_slider_z_size + arm_arm_z_size}" />
   <!-- Arm arms -->
   <xacro:property name="arm_arm_x_size" value="0.04" />

File: debra_description/urdf/debra.urdf (robot description, URDF)
Before this commit: robot debra, 12 links, 11 joints
Links:
- removed link left_arm_support
- removed link right_arm_support
- added link body, mass 0.2; collision box size=0.25 0.25 0.05; visual box size=0.08 0.15 0.3
- link base_link: mass 0.2 -> 0.5
Joints:
- removed joint left_arm_support_joint
- removed joint left_arm_support_left_arm_slider_joint
- removed joint right_arm_support_joint
- removed joint right_arm_support_right_arm_slider_joint
- added joint body_joint: type fixed, parent base_link, child body, origin xyz=0.0                    0.0                    0.175 rpy=0 0 0
- added joint body_left_arm_slider_joint: type prismatic, parent body, child left_arm_slider, origin xyz=0.0                    0.1                    0.14 rpy=0 0 0, axis 0 0 1, limit lower=-0.25 upper=0.0 effort=1000.0 velocity=0.5
- added joint body_right_arm_slider_joint: type prismatic, parent body, child right_arm_slider, origin xyz=0.0                    -0.1                    0.14 rpy=0 0 0, axis 0 0 1, limit lower=-0.25 upper=0.0 effort=1000.0 velocity=0.5

File: debra_description/urdf/debra.xacro (robot description, xacro)
@@ -4,6 +4,6 @@
   <xacro:include filename="$(find debra_description)/urdf/common_properties.xacro" />
   <xacro:include filename="$(find debra_description)/urdf/materials.xacro" />
+  <xacro:include filename="$(find debra_description)/urdf/body.xacro" />
   <xacro:include filename="$(find debra_description)/urdf/wheel.xacro" />
-  <xacro:include filename="$(find debra_description)/urdf/arm_support.xacro" />
   <xacro:include filename="$(find debra_description)/urdf/arm_slider.xacro" />
   <xacro:include filename="$(find debra_description)/urdf/arm_arm.xacro" />
@@ -66,4 +66,9 @@
     <turnGravityOff>false</turnGravityOff>
   </gazebo>
+  <!-- BODY -->
+  <body parent="base_link"
+        translateX="0"
+        translateY="0"
+        flipY="0" />
   <!-- WHEELs -->
   <wheel lr="right"
@@ -78,21 +83,11 @@
          flipY="-1" />
   <!-- ARMS -->
-  <arm_support lr="right"
-               parent="base_link"
-               translateX="0"
-               translateY="-1"
-               flipY="0" />
-  <arm_support lr="left"
-               parent="base_link"
-               translateX="0"
-               translateY="1"
-               flipY="0" />
   <arm_slider lr="right"
-              parent="right_arm_support"
+              parent="body"
               translateX="0"
               translateY="-1"
               flipY="0" />
   <arm_slider lr="left"
-              parent="left_arm_support"
+              parent="body"
               translateX="0"
               translateY="1"
