Commit message: Add laser scanner

File: debra_description/urdf/common_properties.xacro (robot description, xacro)
@@ -80,3 +80,8 @@
   <xacro:property name="arm_forearm_limit_upper" value="${M_PI / 4}" />
   <xacro:property name="arm_forearm_limit_lower" value="${- M_PI / 4}" />
+  <!-- Hokuyo -->
+  <xacro:property name="hokuyo_x_origin_to_parent_origin" value="0.0" />
+  <xacro:property name="hokuyo_y_origin_to_parent_origin" value="0.0" />
+  <xacro:property name="hokuyo_z_origin_to_parent_origin"
+                  value="${(body_z_size + 0.08) / 2}" />
 </robot>

File: debra_description/urdf/debra.urdf (robot description, URDF)
Before this commit: robot debra, 11 links, 10 joints
Links:
- added link hokuyo_link, mass 1e-5; collision box size=0.1 0.1 0.1; visual mesh filename=package://debra_description/meshes/hokuyo.dae
Joints:
- added joint hokuyo_joint: type fixed, parent body, child hokuyo_link, origin xyz=0.0                    0.0                    0.19 rpy=0 0 0

File: debra_description/urdf/debra.xacro (robot description, xacro)
@@ -9,4 +9,5 @@
   <xacro:include filename="$(find debra_description)/urdf/arm_arm.xacro" />
   <xacro:include filename="$(find debra_description)/urdf/arm_forearm.xacro" />
+  <xacro:include filename="$(find debra_description)/urdf/hokuyo.xacro" />
   <!-- BASE-FOOTPRINT -->
   <!-- base_footprint is a fictitious link(frame) that is on the ground right below base_link origin -->
@@ -113,4 +114,6 @@
                translateY="1"
                flipY="0" />
+  <!-- Hokuyo Laser -->
+  <hokuyo parent="body" />
   <!-- Base controller -->
   <gazebo>
@@ -139,39 +142,3 @@
     </plugin>
   </gazebo>
-    <!-- Hokuyo laser controller -->
-  <gazebo reference="hokuyo_link">
-    <sensor type="gpu_ray" name="head_hokuyo_sensor">
-      <pose>0 0 0 0 0 0</pose>
-      <visualize>false</visualize>
-      <update_rate>50</update_rate>
-      <ray>
-        <scan>
-          <horizontal>
-            <samples>720</samples>
-            <resolution>1</resolution>
-            <min_angle>-1.570796</min_angle>
-            <max_angle>1.570796</max_angle>
-          </horizontal>
-        </scan>
-        <range>
-          <min>0.10</min>
-          <max>30.0</max>
-          <resolution>0.01</resolution>
-        </range>
-        <noise>
-          <type>gaussian</type>
-          <!-- Noise parameters based on published spec for Hokuyo laser
-               achieving "+-30mm" accuracy at range < 10m.  A mean of 0.0m and
-               stddev of 0.01m will put 99.7% of samples within 0.03m of the
-               true reading. -->
-          <mean>0.0</mean>
-          <stddev>0.01</stddev>
-        </noise>
-      </ray>
-      <plugin name="gazebo_ros_head_hokuyo_controller" filename="libgazebo_ros_gpu_laser.so">
-        <topicName>/debra/laser/scan</topicName>
-        <frameName>hokuyo_link</frameName>
-      </plugin>
-    </sensor>
-  </gazebo>
 </robot>

Commit message: Update Debra base w/ realistic meshes

File: debra_description/urdf/common_properties.xacro (robot description, xacro)
@@ -38,7 +38,7 @@
   <xacro:property name="wheel_height" value="0.01" />
   <xacro:property name="wheel_mass" value="0.02" /> <!-- in kg -->
-  <xacro:property name="base_x_origin_to_wheel_origin" value="0.0" />
-  <xacro:property name="base_y_origin_to_wheel_origin" value="0.1" />
-  <xacro:property name="base_z_origin_to_wheel_origin" value="-0.01" />
+  <xacro:property name="base_x_origin_to_wheel_origin" value="-0.005" />
+  <xacro:property name="base_y_origin_to_wheel_origin" value="0.078" />
+  <xacro:property name="base_z_origin_to_wheel_origin" value="0.013" />
   <xacro:property name="wheel_separation"
                   value="${base_y_origin_to_wheel_origin * 2}" />

File: debra_description/urdf/debra.urdf (robot description, URDF)
Before this commit: robot debra, 12 links, 11 joints
Links:
- link base_link: mass 0.5 -> 0.546; geometry collision mesh filename=package://debra_description/meshes/base_link.stl; visual mesh filename=package://debra_description/meshes/base_link.stl
- link base_link_left_wheel: mass 0.02 -> 0.066; geometry collision mesh filename=package://debra_description/meshes/wheel.stl; visual mesh filename=package://debra_description/meshes/wheel.stl
- link base_link_right_wheel: mass 0.02 -> 0.066; geometry collision mesh filename=package://debra_description/meshes/wheel.stl; visual mesh filename=package://debra_description/meshes/wheel.stl
Joints:
- joint base_footprint_joint: origin xyz=0 0 0.04 rpy=0 0 0 -> xyz=0 0 0.017 rpy=0 0 0
- joint base_link_left_wheel_joint: origin xyz=0.0                    0.1                    -0.01 rpy=0 0 0 -> xyz=-0.005                    0.078                    0.013 rpy=0 0 0
- joint base_link_right_wheel_joint: origin xyz=0.0                    -0.1                    -0.01 rpy=0 0 0 -> xyz=-0.005                    -0.078                    0.013 rpy=0 0 0

File: debra_description/urdf/debra.xacro (robot description, xacro)
@@ -35,29 +35,31 @@
   <!--Actual body/chassis of the robot-->
   <link name="base_link">
-    <inertial>
-      <mass value="${base_mass}" />
-      <origin xyz="0 0 0"
-              rpy="0 0 0" />
-      <!--The 3x3 rotational inertia matrix. -->
-      <box_inertia m="${base_mass}"
-                   x="${base_x_size}"
-                   y="${base_y_size}"
-                   z="${base_z_size}"/>
-    </inertial>
     <visual>
       <origin xyz="0 0 0"
-              rpy="0 0 0" />
+              rpy="0 0 ${M_PI / 2}" />
       <geometry>
-        <box size="${base_x_size} ${base_y_size} ${base_z_size}"/>
+        <mesh filename="package://debra_description/meshes/base_link.stl" />
       </geometry>
-      <material name="LightGrey" />
+      <material name="base_link_color">
+        <color rgba="0.898 0.918 0.929 1" />
+      </material>
     </visual>
     <collision>
       <origin xyz="0 0 0"
-              rpy="0 0 0 " />
+              rpy="0 0 ${M_PI / 2}" />
       <geometry>
-        <box size="${base_x_size} ${base_y_size} ${base_z_size}"/>
+        <mesh filename="package://debra_description/meshes/base_link.stl" />
       </geometry>
     </collision>
+    <inertial>
+      <origin xyz="0 0 0"
+              rpy="0 0 ${M_PI / 2}" />
+      <mass
+        value="0.546" />
+      <inertia
+        ixx="2.024E-03" ixy="2.367E-07" ixz="-4.520E-06"
+        iyy="3.561E-03" iyz="-4.595E-06"
+        izz="1.834E-03" />
+    </inertial>
   </link>
   <gazebo reference="base_link">
@@ -82,5 +84,5 @@
          translateX="1"
          translateY="1"
-         flipY="-1" />
+         flipY="1" />
   <!-- ARMS -->
   <arm_slider lr="right"

File: debra_description/urdf/wheel.xacro (robot description, xacro)
@@ -11,25 +11,26 @@
       <visual>
         <origin xyz="0 0 0"
-                rpy="${flipY * M_PI / 2} 0 0" />
+                rpy="0 ${(flipY - 1) * M_PI / 2} ${M_PI / 2}" />
         <geometry>
-          <cylinder length="${wheel_height}"
-                    radius="${wheel_radius}" />
+          <mesh filename="package://debra_description/meshes/wheel.stl" />
         </geometry>
-        <material name="DarkGrey" />
+        <material name="wheel_color">
+          <color rgba="0.867 0.910 1 1" />
+        </material>
       </visual>
       <collision>
         <origin xyz="0 0 0"
-                rpy="${flipY * M_PI / 2} 0 0" />
+                rpy="0 ${(flipY - 1) * M_PI / 2} ${M_PI / 2}" />
         <geometry>
-          <cylinder length="${wheel_height}" radius="${wheel_radius}" />
+          <mesh filename="package://debra_description/meshes/wheel.stl" />
         </geometry>
       </collision>
-      <inertial>
-        <mass value="${wheel_mass}" />
+       <inertial>
         <origin xyz="0 0 0"
-                rpy="0 0 0" />
-        <cylinder_inertia  m="${wheel_mass}"
-                           r="${wheel_radius}"
-                           h="${wheel_height}" />
+                rpy="0 ${(flipY - 1) * M_PI / 2} ${M_PI / 2}" />
+        <mass value="0.066" />
+        <inertia ixx="1.234E-05" ixy="-4.969E-22" ixz="-1.613E-23"
+                 iyy="4.849E-22" iyz="-6.502E-06"
+                 izz="3.112E-22" />
       </inertial>
     </link>

Commit message: Collapsing problem solved for armless debra
- Back to base & body configuration on Debra. Body adds enough inertia to avoid robot collapsing
- Needs some optimisation for the collision meshes (use convex meshes) to accelerate collision checks.
- Also need to get the arms back and running on Debra

File: debra_description/urdf/common_properties.xacro (robot description, xacro)
@@ -27,5 +27,5 @@
   <xacro:property name="body_x_size" value="0.08" />
   <xacro:property name="body_y_size"
-                  value="${base_y_size - 2 * arm_slider_y_size}" />
+                  value="${base_y_size - 2 * 0.05}" />
   <xacro:property name="body_z_size" value="0.30" />
   <xacro:property name="body_mass" value="0.2" />
@@ -40,44 +40,7 @@
   <xacro:property name="base_x_origin_to_wheel_origin" value="-0.005" />
   <xacro:property name="base_y_origin_to_wheel_origin" value="0.078" />
-  <xacro:property name="base_z_origin_to_wheel_origin" value="0.013" />
+  <xacro:property name="base_z_origin_to_wheel_origin" value="0.0" />
   <xacro:property name="wheel_separation"
                   value="${base_y_origin_to_wheel_origin * 2}" />
-  <!-- Arm sliders -->
-  <xacro:property name="arm_slider_x_size" value="0.05" />
-  <xacro:property name="arm_slider_y_size" value="0.05" />
-  <xacro:property name="arm_slider_z_size" value="0.02" />
-  <xacro:property name="arm_slider_mass" value="0.01" />
-  <xacro:property name="arm_slider_x_origin_to_base_origin" value="0.0" />
-  <xacro:property name="arm_slider_y_origin_to_base_origin"
-                  value="${(body_y_size + arm_slider_y_size) / 2}" />
-  <xacro:property name="arm_slider_z_origin_to_base_origin"
-                  value="${(body_z_size - arm_slider_z_size) / 2}" />
-  <xacro:property name="arm_slider_limit_upper" value="0.0" />
-  <xacro:property name="arm_slider_limit_lower"
-                  value="${- body_z_size + arm_slider_z_size + arm_arm_z_size}" />
-  <!-- Arm arms -->
-  <xacro:property name="arm_arm_x_size" value="0.04" />
-  <xacro:property name="arm_arm_y_size" value="0.20" />
-  <xacro:property name="arm_arm_z_size" value="0.03" />
-  <xacro:property name="arm_arm_mass" value="0.1" />
-  <xacro:property name="arm_arm_x_origin_to_base_origin" value="0.0" />
-  <xacro:property name="arm_arm_y_origin_to_base_origin"
-                  value="${(arm_arm_y_size + arm_slider_y_size) / 2 - 0.04}" />
-  <xacro:property name="arm_arm_z_origin_to_base_origin"
-                  value="${- (arm_slider_z_size + arm_arm_z_size) / 2}" />
-  <xacro:property name="arm_arm_limit_upper" value="${M_PI / 4}" />
-  <xacro:property name="arm_arm_limit_lower" value="${- M_PI / 4}" />
-  <!-- Arm forearms -->
-  <xacro:property name="arm_forearm_x_size" value="0.04" />
-  <xacro:property name="arm_forearm_y_size" value="0.20" />
-  <xacro:property name="arm_forearm_z_size" value="0.03" />
-  <xacro:property name="arm_forearm_mass" value="0.1" />
-  <xacro:property name="arm_forearm_x_origin_to_base_origin" value="0.0" />
-  <xacro:property name="arm_forearm_y_origin_to_base_origin"
-                  value="${(arm_arm_y_size + arm_forearm_y_size) / 2 - 0.04}" />
-  <xacro:property name="arm_forearm_z_origin_to_base_origin"
-                  value="${- (arm_arm_z_size + arm_forearm_z_size) / 2}" />
-  <xacro:property name="arm_forearm_limit_upper" value="${M_PI / 4}" />
-  <xacro:property name="arm_forearm_limit_lower" value="${- M_PI / 4}" />
   <!-- Hokuyo -->
   <xacro:property name="hokuyo_x_origin_to_parent_origin" value="0.0" />

File: debra_description/urdf/debra.urdf (robot description, URDF)
Before this commit: robot debra, 6 links, 5 joints
Joints:
- joint base_footprint_joint: origin xyz=0 0 0.017 rpy=0 0 0 -> xyz=0 0 0.03 rpy=0 0 0
- joint base_link_left_wheel_joint: origin xyz=-0.005                    0.078                    0.013 rpy=0 0 0 -> xyz=-0.005                    0.078                    0.0 rpy=0 0 0
- joint base_link_right_wheel_joint: origin xyz=-0.005                    -0.078                    0.013 rpy=0 0 0 -> xyz=-0.005                    -0.078                    0.0 rpy=0 0 0

File: debra_description/urdf/debra.xacro (robot description, xacro)
@@ -6,7 +6,4 @@
   <xacro:include filename="$(find debra_description)/urdf/body.xacro" />
   <xacro:include filename="$(find debra_description)/urdf/wheel.xacro" />
-  <xacro:include filename="$(find debra_description)/urdf/arm_slider.xacro" />
-  <xacro:include filename="$(find debra_description)/urdf/arm_arm.xacro" />
-  <xacro:include filename="$(find debra_description)/urdf/arm_forearm.xacro" />
   <xacro:include filename="$(find debra_description)/urdf/hokuyo.xacro" />
   <!-- BASE-FOOTPRINT -->

Commit message: Simplify Debra model: back to a wheelbase with Lidar

File: debra_description/urdf/common_properties.xacro (robot description, xacro)
@@ -24,14 +24,4 @@
   <xacro:property name="base_z_size" value="0.05" />
   <xacro:property name="base_mass" value="0.5" /> <!-- in kg-->
-  <!-- Body -->
-  <xacro:property name="body_x_size" value="0.08" />
-  <xacro:property name="body_y_size"
-                  value="${base_y_size - 2 * 0.05}" />
-  <xacro:property name="body_z_size" value="0.30" />
-  <xacro:property name="body_mass" value="0.2" />
-  <xacro:property name="body_x_origin_to_base_origin" value="0.0" />
-  <xacro:property name="body_y_origin_to_base_origin" value="0.0" />
-  <xacro:property name="body_z_origin_to_base_origin"
-                  value="${(body_z_size + base_z_size) / 2}" />
   <!-- Wheels -->
   <xacro:property name="wheel_radius" value="0.03" />
@@ -47,4 +37,4 @@
   <xacro:property name="hokuyo_y_origin_to_parent_origin" value="0.0" />
   <xacro:property name="hokuyo_z_origin_to_parent_origin"
-                  value="${(body_z_size + 0.08) / 2}" />
+                  value="${(base_z_size + 0.08) / 2}" />
 </robot>

File: debra_description/urdf/debra.urdf (robot description, URDF)
Before this commit: robot debra, 6 links, 5 joints
Links:
- removed link body
Joints:
- removed joint body_joint
- joint hokuyo_joint: origin xyz=0.0                    0.0                    0.19 rpy=0 0 0 -> xyz=0.0                    0.0                    0.065 rpy=0 0 0; parent body -> base_link

File: debra_description/urdf/debra.xacro (robot description, xacro)
@@ -4,5 +4,4 @@
   <xacro:include filename="$(find debra_description)/urdf/common_properties.xacro" />
   <xacro:include filename="$(find debra_description)/urdf/materials.xacro" />
-  <xacro:include filename="$(find debra_description)/urdf/body.xacro" />
   <xacro:include filename="$(find debra_description)/urdf/wheel.xacro" />
   <xacro:include filename="$(find debra_description)/urdf/hokuyo.xacro" />
@@ -66,9 +65,4 @@
     <turnGravityOff>false</turnGravityOff>
   </gazebo>
-  <!-- BODY -->
-  <body parent="base_link"
-        translateX="0"
-        translateY="0"
-        flipY="0" />
   <!-- WHEELs -->
   <wheel lr="right"
@@ -83,5 +77,5 @@
          flipY="1" />
   <!-- Hokuyo Laser -->
-  <hokuyo parent="body" />
+  <hokuyo parent="base_link" />
   <!-- Base controller -->
   <gazebo>

Commit message: Fix wheels on Debra model

File: debra_description/urdf/common_properties.xacro (robot description, xacro)
@@ -22,6 +22,6 @@
   <xacro:property name="base_x_size" value="0.25" />
   <xacro:property name="base_y_size" value="0.25" />
-  <xacro:property name="base_z_size" value="0.05" />
-  <xacro:property name="base_mass" value="0.5" /> <!-- in kg-->
+  <xacro:property name="base_z_size" value="0.0413" />
+  <xacro:property name="base_mass" value="0.55" /> <!-- in kg-->
   <!-- Wheels -->
   <xacro:property name="wheel_radius" value="0.03" />
@@ -30,5 +30,5 @@
   <xacro:property name="base_x_origin_to_wheel_origin" value="-0.005" />
   <xacro:property name="base_y_origin_to_wheel_origin" value="0.078" />
-  <xacro:property name="base_z_origin_to_wheel_origin" value="0.0" />
+  <xacro:property name="base_z_origin_to_wheel_origin" value="0.015" />
   <xacro:property name="wheel_separation"
                   value="${base_y_origin_to_wheel_origin * 2}" />

File: debra_description/urdf/debra.urdf (robot description, URDF)
Before this commit: robot debra, 5 links, 4 joints
Joints:
- joint base_footprint_joint: origin xyz=0 0 0.03 rpy=0 0 0 -> xyz=0 0 0.015 rpy=0 0 0
- joint base_link_left_wheel_joint: origin xyz=-0.005                    0.078                    0.0 rpy=0 0 0 -> xyz=-0.005                    0.078                    0.015 rpy=0 0 0
- joint base_link_right_wheel_joint: origin xyz=-0.005                    -0.078                    0.0 rpy=0 0 0 -> xyz=-0.005                    -0.078                    0.015 rpy=0 0 0
- joint hokuyo_joint: origin xyz=0.0                    0.0                    0.065 rpy=0 0 0 -> xyz=0.0                    0.0                    0.06065 rpy=0 0 0
