Commit message: Switch from car config to differential drive

File: debra_description/urdf/debra.urdf (robot description, URDF)
Before this commit: robot debra, 5 links, 4 joints
Links:
- removed link b_l_wheel
- removed link b_r_wheel
- removed link f_l_wheel
- removed link f_r_wheel
- added link base_footprint, mass 0.0001; visual box size=0.001 0.001 0.001
- added link base_link_left_wheel, mass 0.1; collision cylinder length=0.05 radius=0.2; visual cylinder length=0.05 radius=0.2
- added link base_link_right_wheel, mass 0.1; collision cylinder length=0.05 radius=0.2; visual cylinder length=0.05 radius=0.2
- link base_link: mass None -> 1; geometry collision box size=1 0.5 0.25; visual box size=1 0.5 0.25
Joints:
- removed joint joint_b_l_wheel
- removed joint joint_b_r_wheel
- removed joint joint_f_l_wheel
- removed joint joint_f_r_wheel
- added joint base_footprint_joint: type fixed, parent base_footprint, child base_link, origin xyz=0 0 0.3 rpy=0 0 0
- added joint base_link_left_wheel_joint: type continuous, parent base_link, child base_link_left_wheel, origin xyz=0.0                    0.3                    -0.1 rpy=0 0 0, axis 0 1 0, limit effort=100 velocity=100
- added joint base_link_right_wheel_joint: type continuous, parent base_link, child base_link_right_wheel, origin xyz=0.0                    -0.3                    -0.1 rpy=0 0 0, axis 0 1 0, limit effort=100 velocity=100

File: debra_description/urdf/debra.xacro (robot description, xacro)
@@ -2,20 +2,7 @@
 <robot name="debra" xmlns:xacro="http://www.ros.org/wiki/xacro">
   <!-- Included URDF/XACRO Files -->
+  <xacro:include filename="$(find debra_description)/urdf/common_properties.xacro" />
   <xacro:include filename="$(find debra_description)/urdf/materials.xacro" />
   <xacro:include filename="$(find debra_description)/urdf/wheel.xacro" />
-  <!-- PROPERTY LIST -->
-  <!--All units in m-kg-s-radians unit system -->
-  <property name="M_PI" value="3.1415926535897931" />
-  <!-- Main Body-base -->
-  <property name="base_x_size" value="1.0" />
-  <property name="base_y_size" value="0.5" />
-  <property name="base_z_size" value="0.25" />
-  <property name="base_mass" value="35" /> <!-- in kg-->
-  <!--Inertial macros for the box and cylinder. Units are kg*m^2-->
-  <macro name="box_inertia" params="m x y z">
-    <inertia  ixx="${m*(y*y+z*z)/12}" ixy = "0" ixz = "0"
-              iyy="${m*(x*x+z*z)/12}" iyz = "0"
-              izz="${m*(x*x+z*z)/12}" />
-  </macro>
   <!-- BASE-FOOTPRINT -->
   <!-- base_footprint is a fictitious link(frame) that is on the ground right below base_link origin -->
@@ -23,11 +10,13 @@
     <inertial>
       <mass value="0.0001" />
-      <origin xyz="0 0 0" />
+      <origin xyz="0 0 0"
+              rpy="0 0 0"/>
       <inertia ixx="0.0001" ixy="0.0" ixz="0.0"
-          iyy="0.0001" iyz="0.0"
-          izz="0.0001" />
+               iyy="0.0001" iyz="0.0"
+               izz="0.0001" />
     </inertial>
     <visual>
-        <origin xyz="0 0 0" rpy="0 0 0" />
+        <origin xyz="0 0 0"
+                rpy="0 0 0" />
         <geometry>
             <box size="0.001 0.001 0.001" />
@@ -38,6 +27,8 @@
     <turnGravityOff>false</turnGravityOff>
   </gazebo>
-  <joint name="base_footprint_joint" type="fixed">
-  <origin xyz="0 0 ${wheel_radius - base_z_origin_to_wheel_origin}" rpy="0 0 0" />
+  <joint name="base_footprint_joint"
+         type="fixed">
+  <origin xyz="0 0 ${wheel_radius - base_z_origin_to_wheel_origin}"
+          rpy="0 0 0" />
     <parent link="base_footprint"/>
     <child link="base_link" />
@@ -49,10 +40,15 @@
     <inertial>
       <mass value="${base_mass}" />
-      <origin xyz="0 0 0" />
+      <origin xyz="0 0 0"
+              rpy="0 0 0" />
       <!--The 3x3 rotational inertia matrix. -->
-      <box_inertia  m="${base_mass}" x="${base_x_size}" y="${base_y_size}" z="${base_z_size}"/>
+      <box_inertia m="${base_mass}"
+                   x="${base_x_size}"
+                   y="${base_y_size}"
+                   z="${base_z_size}"/>
     </inertial>
     <visual>
-      <origin xyz="0 0 0" rpy="0 0 0" />
+      <origin xyz="0 0 0"
+              rpy="0 0 0" />
       <geometry>
         <box size="1 0.5 0.25"/>
@@ -61,5 +57,6 @@
     </visual>
     <collision>
-      <origin xyz="0 0 0" rpy="0 0 0 " />
+      <origin xyz="0 0 0"
+              rpy="0 0 0 " />
       <geometry>
         <box size="1 0.5 0.25"/>
@@ -72,26 +69,31 @@
   </gazebo>
   <!-- WHEELs -->
-  <wheel fb="front" lr="right" parent="base_link" translateX="1" translateY="-1" flipY="-1"/>
-  <wheel fb="front" lr="left" parent="base_link" translateX="1" translateY="1" flipY="-1"/>
-  <wheel fb="back" lr="right" parent="base_link" translateX="-1" translateY="-1" flipY="-1"/>
-  <wheel fb="back" lr="left" parent="base_link" translateX="-1" translateY="1" flipY="-1"/>
+  <wheel lr="right"
+         parent="base_link"
+         translateX="1"
+         translateY="-1"
+         flipY="-1"/>
+  <wheel lr="left"
+         parent="base_link"
+         translateX="1"
+         translateY="1"
+         flipY="-1"/>
   <gazebo>
-    <plugin name="skid_steer_drive_controller" filename="libgazebo_ros_skid_steer_drive.so">
+    <plugin name="differential_drive_controller"
+            filename="libgazebo_ros_diff_drive.so">
       <alwaysOn>true</alwaysOn>
-      <updateRate>100.0</updateRate>
-      <leftFrontJoint>front_left_wheel_joint</leftFrontJoint>
-      <rightFrontJoint>front_right_wheel_joint</rightFrontJoint>
-      <leftRearJoint>back_left_wheel_joint</leftRearJoint>
-      <rightRearJoint>back_right_wheel_joint</rightRearJoint>
-      <wheelSeparation>${base_y_size}</wheelSeparation>
-      <wheelDiameter>${2*wheel_radius}</wheelDiameter>
-      <torque>35</torque>
-      <broadcastTF>1</broadcastTF>
-      <odometryFrame>map</odometryFrame>
+      <updateRate>${update_rate}</updateRate>
+      <leftJoint>base_link_right_wheel_joint</leftJoint>
+      <rightJoint>base_link_left_wheel_joint</rightJoint>
+      <wheelSeparation>${wheel_separation}</wheelSeparation>
+      <wheelDiameter>${wheel_radius * 2}</wheelDiameter>
+      <torque>20</torque>
       <commandTopic>cmd_vel</commandTopic>
       <odometryTopic>odom</odometryTopic>
+      <odometryFrame>odom</odometryFrame>
       <robotBaseFrame>base_footprint</robotBaseFrame>
     </plugin>
-    <plugin name="gazebo_ros_control" filename="libgazebo_ros_control.so" />
+    <plugin name="gazebo_ros_control"
+            filename="libgazebo_ros_control.so" />
   </gazebo>
 </robot>

File: debra_description/urdf/materials.xacro (robot description, xacro)
@@ -10,8 +10,11 @@
     <color rgba="0.0 0.8 0.0 1.0"/>
   </material>
-  <material name="Gray">
+  <material name="LightGrey">
     <color rgba="0.7 0.7 0.7 1.0"/>
   </material>
-  <material name="DarkGray">
+  <material name="Grey">
+    <color rgba="0.5 0.5 0.5 1.0"/>
+  </material>
+  <material name="DarkGrey">
     <color rgba="0.3 0.3 0.3 1.0"/>
   </material>

File: debra_description/urdf/wheel.xacro (robot description, xacro)
@@ -1,27 +1,24 @@
 <?xml version="1.0"?>
 <robot name="wheel" xmlns:xacro="http://www.ros.org/wiki/xacro">
+  <!-- Included URDF/XACRO Files -->
+  <xacro:include
+    filename="$(find debra_description)/urdf/common_properties.xacro" />
   <!-- Wheels -->
-  <property name="wheel_radius" value="0.2" />
-  <property name="wheel_height" value="0.1" />
-  <property name="wheel_mass" value="2.5" /> <!-- in kg-->
-  <property name="base_x_origin_to_wheel_origin" value="0.25" />
-  <property name="base_y_origin_to_wheel_origin" value="0.3" />
-  <property name="base_z_origin_to_wheel_origin" value="0.0" />
-  <macro name="cylinder_inertia" params="m r h">
-    <inertia  ixx="${m*(3*r*r+h*h)/12}" ixy = "0" ixz = "0"
-              iyy="${m*(3*r*r+h*h)/12}" iyz = "0"
-              izz="${m*r*r/2}" />
-  </macro>
-  <xacro:macro name="wheel" params="fb lr parent translateX translateY flipY"> <!--fb : front, back ; lr: left, right -->
-    <link name="${fb}_${lr}_wheel">
+  <xacro:macro name="wheel"
+               params="lr parent translateX translateY flipY">
+  <!--lr: left, right -->
+    <link name="${parent}_${lr}_wheel">
       <visual>
-        <origin xyz="0 0 0" rpy="${flipY*M_PI/2} 0 0" />
+        <origin xyz="0 0 0"
+                rpy="${flipY * M_PI / 2} 0 0" />
         <geometry>
-          <cylinder length="${wheel_height}" radius="${wheel_radius}" />
+          <cylinder length="${wheel_height}"
+                    radius="${wheel_radius}" />
         </geometry>
-        <material name="DarkGray" />
+        <material name="DarkGrey" />
       </visual>
       <collision>
-        <origin xyz="0 0 0" rpy="${flipY*M_PI/2} 0 0" />
+        <origin xyz="0 0 0"
+                rpy="${flipY * M_PI / 2} 0 0" />
         <geometry>
           <cylinder length="${wheel_height}" radius="${wheel_radius}" />
@@ -30,9 +27,12 @@
       <inertial>
         <mass value="${wheel_mass}" />
-        <origin xyz="0 0 0" />
-        <cylinder_inertia  m="${wheel_mass}" r="${wheel_radius}" h="${wheel_height}" />
+        <origin xyz="0 0 0"
+                rpy="0 0 0" />
+        <cylinder_inertia  m="${wheel_mass}"
+                           r="${wheel_radius}"
+                           h="${wheel_height}" />
       </inertial>
     </link>
-    <gazebo reference="${fb}_${lr}_wheel">
+    <gazebo reference="${parent}_${lr}_wheel">
       <mu1 value="1.0"/>
       <mu2 value="1.0"/>
@@ -43,18 +43,25 @@
       <turnGravityOff>false</turnGravityOff>
     </gazebo>
-    <joint name="${fb}_${lr}_wheel_joint" type="continuous">
+    <joint name="${parent}_${lr}_wheel_joint"
+           type="continuous">
       <parent link="${parent}"/>
-      <child link="${fb}_${lr}_wheel"/>
+      <child link="${parent}_${lr}_wheel"/>
       <hardwareInterface>EffortJointInterface</hardwareInterface>
-      <origin xyz="${translateX * base_x_origin_to_wheel_origin} ${translateY * base_y_origin_to_wheel_origin} ${base_z_origin_to_wheel_origin}" rpy="0 0 0" />
-      <axis xyz="0 1 0" rpy="0 0 0" />
-      <limit effort="100" velocity="100"/>
-      <joint_properties damping="0.0" friction="0.0"/>
+      <origin xyz="${translateX * base_x_origin_to_wheel_origin}
+                   ${translateY * base_y_origin_to_wheel_origin}
+                   ${base_z_origin_to_wheel_origin}"
+              rpy="0 0 0" />
+      <axis xyz="0 1 0"
+            rpy="0 0 0" />
+      <limit effort="100"
+             velocity="100"/>
+      <joint_properties damping="0.0"
+                        friction="0.0"/>
     </joint>
     <!-- Transmission is important to link the joints and the controller -->
-    <transmission name="${fb}_${lr}_wheel_joint_trans">
+    <transmission name="${parent}_${lr}_wheel_joint_trans">
       <type>transmission_interface/SimpleTransmission</type>
-      <joint name="${fb}_${lr}_wheel_joint" />
-      <actuator name="${fb}_${lr}_wheel_joint_motor">
+      <joint name="${parent}_${lr}_wheel_joint" />
+      <actuator name="${parent}_${lr}_wheel_joint_motor">
         <hardwareInterface>EffortJointInterface</hardwareInterface>
         <mechanicalReduction>1</mechanicalReduction>

Commit message: Robot w/ base only not collapsing but not moving properly either (oscillating)

File: debra_description/urdf/debra.urdf (robot description, URDF)
Before this commit: robot debra, 12 links, 11 joints
Links:
- removed link left_arm_arm
- removed link left_arm_forearm
- removed link left_arm_slider
- removed link right_arm_arm
- removed link right_arm_forearm
- removed link right_arm_slider
Joints:
- removed joint body_left_arm_slider_joint
- removed joint body_right_arm_slider_joint
- removed joint left_arm_arm_left_arm_forearm_joint
- removed joint left_arm_slider_left_arm_arm_joint
- removed joint right_arm_arm_right_arm_forearm_joint
- removed joint right_arm_slider_right_arm_arm_joint

File: debra_description/urdf/debra.xacro (robot description, xacro)
@@ -58,7 +58,7 @@
         value="0.546" />
       <inertia
-        ixx="2.024E-03" ixy="2.367E-07" ixz="-4.520E-06"
-        iyy="3.561E-03" iyz="-4.595E-06"
-        izz="1.834E-03" />
+        ixx="0.1" ixy="0.0" ixz="0.0"
+        iyy="0.1" iyz="0.0"
+        izz="0.1" />
     </inertial>
   </link>
@@ -85,35 +85,4 @@
          translateY="1"
          flipY="1" />
-  <!-- ARMS -->
-  <arm_slider lr="right"
-              parent="body"
-              translateX="0"
-              translateY="-1"
-              flipY="0" />
-  <arm_slider lr="left"
-              parent="body"
-              translateX="0"
-              translateY="1"
-              flipY="0" />
-  <arm_arm lr="right"
-           parent="right_arm_slider"
-           translateX="0"
-           translateY="-1"
-           flipY="0" />
-  <arm_arm lr="left"
-           parent="left_arm_slider"
-           translateX="0"
-           translateY="1"
-           flipY="0" />
-  <arm_forearm lr="right"
-               parent="right_arm_arm"
-               translateX="0"
-               translateY="-1"
-               flipY="0" />
-  <arm_forearm lr="left"
-               parent="left_arm_arm"
-               translateX="0"
-               translateY="1"
-               flipY="0" />
   <!-- Hokuyo Laser -->
   <hokuyo parent="body" />

File: debra_description/urdf/wheel.xacro (robot description, xacro)
@@ -30,7 +30,7 @@
                 rpy="0 ${(flipY - 1) * M_PI / 2} ${M_PI / 2}" />
         <mass value="0.066" />
-        <inertia ixx="1.234E-05" ixy="-4.969E-22" ixz="-1.613E-23"
-                 iyy="4.849E-22" iyz="-6.502E-06"
-                 izz="3.112E-22" />
+        <inertia ixx="0.1" ixy="0.0" ixz="0.0"
+                 iyy="0.1" iyz="0.0"
+                 izz="0.1" />
       </inertial>
     </link>

Commit message: Use Sick lidar (tim561) instead of Hokuyo

File: debra_description/urdf/debra.urdf (robot description, URDF)
Before this commit: robot debra, 5 links, 4 joints
Links:
- removed link hokuyo_link
- added link laser, mass 0.25; collision mesh filename=package://sick_tim/meshes/sick_tim551.stl; visual mesh filename=package://sick_tim/meshes/sick_tim551.stl
Joints:
- removed joint hokuyo_joint
- added joint base_link_laser_joint: type fixed, parent base_link, child laser, origin xyz=0 0 0.06296 rpy=0 0 0
- joint base_link_left_wheel_joint: limit effort=100 velocity=100 -> effort=10 velocity=2
- joint base_link_right_wheel_joint: limit effort=100 velocity=100 -> effort=10 velocity=2

File: debra_description/urdf/debra.xacro (robot description, xacro)
@@ -5,5 +5,5 @@
   <xacro:include filename="$(find debra_description)/urdf/materials.xacro" />
   <xacro:include filename="$(find debra_description)/urdf/wheel.xacro" />
-  <xacro:include filename="$(find debra_description)/urdf/hokuyo.xacro" />
+  <xacro:include filename="$(find sick_tim)/urdf/sick_tim_56x.urdf.xacro" />
   <!-- BASE-FOOTPRINT -->
   <!-- base_footprint is a fictitious link(frame) that is on the ground right below base_link origin -->
@@ -13,5 +13,5 @@
                 rpy="0 0 0" />
         <geometry>
-            <box size="0.001 0.001 0.001" />
+          <box size="0.001 0.001 0.001" />
         </geometry>
     </visual>
@@ -38,5 +38,5 @@
       </geometry>
       <material name="base_link_color">
-        <color rgba="0.898 0.918 0.929 1" />
+        <color rgba="0.9 0.9 0.9 1.0" />
       </material>
     </visual>
@@ -76,31 +76,5 @@
          translateY="1"
          flipY="1" />
-  <!-- Hokuyo Laser -->
-  <hokuyo parent="base_link" />
-  <!-- Base controller -->
-  <gazebo>
-    <plugin name="differential_drive_controller"
-            filename="libgazebo_ros_diff_drive.so">
-      <alwaysOn>true</alwaysOn>
-      <updateRate>${update_rate}</updateRate>
-      <leftJoint>base_link_right_wheel_joint</leftJoint>
-      <rightJoint>base_link_left_wheel_joint</rightJoint>
-      <wheelSeparation>${wheel_separation}</wheelSeparation>
-      <wheelDiameter>${wheel_radius * 2}</wheelDiameter>
-      <torque>20</torque>
-      <commandTopic>cmd_vel</commandTopic>
-      <odometryTopic>odom</odometryTopic>
-      <odometryFrame>odom</odometryFrame>
-      <robotBaseFrame>base_footprint</robotBaseFrame>
-    </plugin>
-    <plugin name="gazebo_ros_control"
-            filename="libgazebo_ros_control.so" />
-  </gazebo>
-  <!-- Arm controller -->
-  <gazebo>
-    <plugin name="gazebo_ros_control"
-            filename="libgazebo_ros_control.so">
-      <robotNamespace>/debra</robotNamespace>
-    </plugin>
-  </gazebo>
+  <!-- Sick Lidar Tim561 -->
+  <xacro:sick_tim561 name="laser" ros_topic="scan" parent="base_link" />
 </robot>

File: debra_description/urdf/wheel.xacro (robot description, xacro)
@@ -15,6 +15,6 @@
           <mesh filename="package://debra_description/meshes/wheel.stl" />
         </geometry>
-        <material name="wheel_color">
-          <color rgba="0.867 0.910 1 1" />
+        <material name="Yellow">
+          <color rgba="1 1 0 1" />
         </material>
       </visual>
@@ -38,8 +38,8 @@
       <mu1 value="1.0"/>
       <mu2 value="1.0"/>
-      <kp  value="10000000.0" />
-      <kd  value="1.0" />
+      <kp  value="0.0" />
+      <kd  value="0.0" />
       <fdir1 value="1 0 0"/>
-      <material>Gazebo/Blue</material>
+      <material>Gazebo/Yellow</material>
       <turnGravityOff>false</turnGravityOff>
     </gazebo>
@@ -55,6 +55,6 @@
       <axis xyz="0 1 0"
             rpy="0 0 0" />
-      <limit effort="100"
-             velocity="100"/>
+      <limit effort="10"
+             velocity="2"/>
       <joint_properties damping="0.0"
                         friction="0.0"/>
