Commit message: Debra base with lidar functional
Publish tf / joint states correctly (so the robot doesn't collapse)
Force visualisation of lidar ray
Minor color corrections

File: debra_description/urdf/debra.xacro (robot description, xacro)
@@ -37,7 +37,5 @@
         <mesh filename="package://debra_description/meshes/base_link.stl" />
       </geometry>
-      <material name="base_link_color">
-        <color rgba="0.9 0.9 0.9 1.0" />
-      </material>
+      <material name="White"/>
     </visual>
     <collision>

File: debra_description/urdf/wheel.xacro (robot description, xacro)
@@ -15,7 +15,5 @@
           <mesh filename="package://debra_description/meshes/wheel.stl" />
         </geometry>
-        <material name="Yellow">
-          <color rgba="1 1 0 1" />
-        </material>
+        <material name="Yellow"/>
       </visual>
       <collision>
