Commit message: Gazebo controllers removed

File: debra_description/urdf/wheel.xacro (robot description, xacro)
@@ -55,18 +55,6 @@
       <limit effort="10"
              velocity="2"/>
-      <joint_properties damping="0.0"
-                        friction="0.0"/>
+      <joint_properties damping="0.0" friction="0.0"/>
     </joint>
-    <!-- Transmission is important to link the joints and the controller -->
-    <transmission name="${parent}_${lr}_wheel_joint_trans">
-      <type>transmission_interface/SimpleTransmission</type>
-      <joint name="${parent}_${lr}_wheel_joint">
-        <hardwareInterface>EffortJointInterface</hardwareInterface>
-      </joint>
-      <actuator name="${parent}_${lr}_wheel_joint_motor">
-        <hardwareInterface>EffortJointInterface</hardwareInterface>
-        <mechanicalReduction>1</mechanicalReduction>
-      </actuator>
-    </transmission>
   </xacro:macro>
 </robot>
